File: 3dprinter.kicad_pcb (KiCad board)
At the start: 2 copper layers, 148.1 x 75 mm, 108 parts, among them J1 6P IDC CONNECTOR, J10 MCU_PROG, J11 Conn_01x04, J12 MCU_PROG, J13 Conn_01x04, J14 MCU_PROG, J15 Conn_01x04, J16 MCU_PROG, J17 Conn_02x04_Odd_Even, J18 Conn_01x18, J2 USB_B_Micro, J3 Conn_01x02, J4 X_END, J5 Thermistor, J6 Y_END, J7 Z_END, J8 Heaters & Fans, J9 Conn_01x04, Q1 Mos, Q2 Mos, Q3 Mos, SW1 6x6 SMD, U1 ATmega2560-16A, U2 FT232RL, U3 L7805, Y1 16MHz

Commit message: finish
Parts:
- added G***: LOGO, M3FOOTPRINT:ironmanmask, F.Cu at (175.9, 84.6)
- added G***: LOGO, M3FOOTPRINT:arcreactor, F.Cu at (172.7, 95.4)
- added G***: LOGO, M3FOOTPRINT:ironman, F.Cu at (230.4, 73.7)
- C1, C2, C3, C4, C5, C6, C7: footprint Capacitor_SMD:C_0805_2012Metric_Pad1.18x1.45mm_HandSolder -> Capacitor_SMD:C_0805_2012Metric
- D1, D2, D3: footprint LED_SMD:LED_0805_2012Metric_Pad1.15x1.40mm_HandSolder -> LED_SMD:LED_0805_2012Metric
- R1, R2, R39, R4, R40, R41, R42, R43, R44, R5: footprint Resistor_SMD:R_0805_2012Metric_Pad1.20x1.40mm_HandSolder -> Resistor_SMD:R_0805_2012Metric
- moved R9 71.8 mm to (136.2, 104.0)
- moved R16 71.8 mm to (143.8, 104.0)
- moved R20 71.8 mm to (151.5, 104.0)
- moved C10 68.7 mm to (147.6, 104.6)
- moved C11 68.7 mm to (155.2, 104.6)
- moved C9 68.7 mm to (140.0, 104.6)
- moved J5 68.5 mm to (136.1, 117.8)
- moved J1 40.2 mm to (194.5, 97.6), turned to 90 degrees
- moved C8 29.1 mm to (221.1, 83.1)
- moved R1 29.1 mm to (211.5, 84.0)
- moved R8 29.1 mm to (214.5, 83.1)
- moved SW1 29.1 mm to (217.8, 87.6)
- moved Y1 24.3 mm to (185.9, 85.7), turned to 135 degrees
- moved J4 23.0 mm to (158.9, 117.8)
- moved J6 23.0 mm to (181.8, 117.8)
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Connections:
- C11 pad 1: THERM2 -> THERM0
- C9 pad 1: THERM0 -> THERM2
- J1 pad 2: +5V -> RES
- J1 pad 3: SCK -> MOSI
- J1 pad 4: MOSI -> +5V
- J1 pad 5: RES -> SCK
- J5 pad 2: THERM0 -> THERM2
- J5 pad 6: THERM2 -> THERM0
- R16 pad 2: VCC -> +5V
- R20 pad 1: THERM2 -> THERM0
- R20 pad 2: VCC -> +5V
- R9 pad 1: THERM0 -> THERM2
- R9 pad 2: VCC -> +5V
- U1 pad 17: unconnected-(U1-Pad17) -> D8
- U1 pad 18: unconnected-(U1-Pad18) -> D9
- U1 pad 23: unconnected-(U1-Pad23) -> D10
- U1 pad 40: D44 -> unconnected-(U1-Pad40)
- U1 pad 42: D42 -> unconnected-(U1-Pad42)
- U1 pad 43: SCL -> unconnected-(U1-Pad43)
- U1 pad 44: SDA -> unconnected-(U1-Pad44)
- U1 pad 52: D40 -> unconnected-(U1-Pad52)
- U1 pad 78: D22 -> unconnected-(U1-Pad78)
- U1 pad 85: A12 -> unconnected-(U1-Pad85)
- U1 pad 86: A11 -> unconnected-(U1-Pad86)
- U1 pad 87: A10 -> unconnected-(U1-Pad87)
- U1 pad 88: A9 -> unconnected-(U1-Pad88)
- U1 pad 92: A5 -> unconnected-(U1-Pad92)
- U1 pad 93: A4 -> unconnected-(U1-Pad93)
- U1 pad 94: A3 -> unconnected-(U1-Pad94)
Routing:
- net +5V: track 391.4 -> 638.4 mm, vias 5 -> 17
- net D29: track 0.00 -> 155.9 mm, vias 0 -> 2
- net D27: track 0.00 -> 149.7 mm, vias 0 -> 2
- net D23: track 0.00 -> 144.0 mm, vias 0 -> 2
- net D25: track 0.00 -> 143.2 mm
- net D8: track 1.80 -> 138.0 mm, vias 0 -> 4
- net D31: track 0.00 -> 128.8 mm, vias 0 -> 3
- net D33: track 0.00 -> 126.9 mm, vias 0 -> 3
- net D35: track 0.00 -> 126.8 mm, vias 0 -> 3
- net D32: track 0.00 -> 126.6 mm, vias 0 -> 3
- net D37: track 0.00 -> 124.0 mm, vias 0 -> 3
- net D9: track 1.80 -> 120.9 mm, vias 0 -> 4
- net D16: track 0.00 -> 102.2 mm, vias 0 -> 2
- net D17: track 0.00 -> 100.9 mm, vias 0 -> 2
- net D10: track 1.80 -> 90.6 mm, vias 0 -> 2
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Other:
- outline, holes or cut-outs redrawn
- board text added: "+5V"
- board text added: "GND"
- board text added: "TEMP0"
- board text added: "TEMP1"
- board text added: "TEMP2"
- board text added: "XMAX"
- board text added: "XMIN"
- board text added: "YMAX"
- board text added: "YMIN"
- board text added: "ZMAX"
- board text added: "ZMIN"
