File: FT232.kicad_sch (KiCad schematic)
At the start: 13 parts

Commit message: PCB
Parts:
- gave numbers to parts that had none: 13
Changed lines of the file:
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@@
   (symbol (lib_id "Device:R_Small_US") (at 105.41 60.96 90) (unit 1)
     (in_bom yes) (on_board yes)
-    (property "Reference" "R?" (id 0) (at 103.505 62.865 90))
+    (property "Reference" "R36" (id 0) (at 103.505 62.865 90))
     (property "Value" "330R" (id 1) (at 107.95 62.865 90))
     (property "Footprint" "Resistor_SMD:R_0805_2012Metric" (id 2) (at 105.41 60.96 0)
@@
   (symbol (lib_id "power:+5V") (at 110.49 53.34 0) (unit 1)
     (in_bom yes) (on_board yes) (fields_autoplaced)
-    (property "Reference" "#PWR?" (id 0) (at 110.49 57.15 0)
+    (property "Reference" "#PWR067" (id 0) (at 110.49 57.15 0)
       (effects (font (size 1.27 1.27)) hide)
     )
@@
   (symbol (lib_id "power:+5V") (at 71.12 20.955 0) (unit 1)
     (in_bom yes) (on_board yes)
-    (property "Reference" "#PWR?" (id 0) (at 71.12 24.765 0)
+    (property "Reference" "#PWR065" (id 0) (at 71.12 24.765 0)
       (effects (font (size 1.27 1.27)) hide)
     )
@@
   (symbol (lib_id "Device:LED_Small") (at 96.52 60.96 0) (unit 1)
     (in_bom yes) (on_board yes)
-    (property "Reference" "D?" (id 0) (at 99.06 59.69 0))
+    (property "Reference" "D11" (id 0) (at 99.06 59.69 0))
     (property "Value" "LED_RED" (id 1) (at 96.52 62.865 0))
     (property "Footprint" "LED_SMD:LED_0805_2012Metric" (id 2) (at 96.52 60.96 90)
@@
   (symbol (lib_id "Device:LED_Small") (at 96.52 54.61 0) (unit 1)
     (in_bom yes) (on_board yes)
-    (property "Reference" "D?" (id 0) (at 99.06 53.34 0))
+    (property "Reference" "D10" (id 0) (at 99.06 53.34 0))
     (property "Value" "LED_RED" (id 1) (at 96.52 56.515 0))
     (property "Footprint" "LED_SMD:LED_0805_2012Metric" (id 2) (at 96.52 54.61 90)
@@
   (symbol (lib_id "Device:R_Small_US") (at 99.06 38.1 90) (unit 1)
     (in_bom yes) (on_board yes)
-    (property "Reference" "R?" (id 0) (at 97.155 40.005 90))
+    (property "Reference" "R31" (id 0) (at 97.155 40.005 90))
     (property "Value" "100R_NM" (id 1) (at 104.14 40.005 90))
     (property "Footprint" "Resistor_SMD:R_0805_2012Metric" (id 2) (at 99.06 38.1 0)
@@
   (symbol (lib_id "power:GNDREF") (at 72.39 80.645 0) (unit 1)
     (in_bom yes) (on_board yes) (fields_autoplaced)
-    (property "Reference" "#PWR?" (id 0) (at 72.39 86.995 0)
+    (property "Reference" "#PWR066" (id 0) (at 72.39 86.995 0)
       (effects (font (size 1.27 1.27)) hide)
     )
@@
   (symbol (lib_id "Device:R_Small_US") (at 100.965 33.02 90) (unit 1)
     (in_bom yes) (on_board yes)
-    (property "Reference" "R?" (id 0) (at 99.06 34.29 90)
+    (property "Reference" "R33" (id 0) (at 99.06 34.29 90)
       (effects (font (size 1.27 1.27)) (justify left))
     )
@@
   (symbol (lib_id "Device:R_Small_US") (at 105.41 54.61 90) (unit 1)
     (in_bom yes) (on_board yes)
-    (property "Reference" "R?" (id 0) (at 103.505 56.515 90))
+    (property "Reference" "R35" (id 0) (at 103.505 56.515 90))
     (property "Value" "330R" (id 1) (at 107.95 56.515 90))
     (property "Footprint" "Resistor_SMD:R_0805_2012Metric" (id 2) (at 105.41 54.61 0)
@@
   (symbol (lib_id "power:+5V") (at 39.37 43.18 0) (unit 1)
     (in_bom yes) (on_board yes)
-    (property "Reference" "#PWR?" (id 0) (at 39.37 46.99 0)
+    (property "Reference" "#PWR064" (id 0) (at 39.37 46.99 0)
       (effects (font (size 1.27 1.27)) hide)
     )
@@
   (symbol (lib_id "Device:R_Small_US") (at 99.06 43.18 90) (unit 1)
     (in_bom yes) (on_board yes)
-    (property "Reference" "R?" (id 0) (at 97.155 45.085 90))
+    (property "Reference" "R32" (id 0) (at 97.155 45.085 90))
     (property "Value" "100R_NM or 100nF" (id 1) (at 107.95 45.085 90))
     (property "Footprint" "Resistor_SMD:R_0805_2012Metric" (id 2) (at 99.06 43.18 0)
@@
   (symbol (lib_id "Device:C_Small") (at 41.91 33.02 270) (unit 1)
     (in_bom yes) (on_board yes)
-    (property "Reference" "C?" (id 0) (at 41.91 35.56 90))
+    (property "Reference" "C21" (id 0) (at 41.91 35.56 90))
     (property "Value" "100nF" (id 1) (at 41.91 30.48 90))
     (property "Footprint" "Capacitor_SMD:C_0805_2012Metric" (id 2) (at 41.91 33.02 0)
@@
   (symbol (lib_id "Device:C_Small") (at 46.355 27.305 180) (unit 1)
     (in_bom yes) (on_board yes)
-    (property "Reference" "C?" (id 0) (at 43.815 27.305 90))
+    (property "Reference" "C22" (id 0) (at 43.815 27.305 90))
     (property "Value" "100nF" (id 1) (at 51.435 27.305 0))
     (property "Footprint" "Capacitor_SMD:C_0805_2012Metric" (id 2) (at 46.355 27.305 0)
@@
   (symbol (lib_id "Interface_USB:FT232RL") (at 71.12 50.8 0) (unit 1)
     (in_bom yes) (on_board yes) (fields_autoplaced)
-    (property "Reference" "U?" (id 0) (at 75.6794 23.495 0)
+    (property "Reference" "U2" (id 0) (at 75.6794 23.495 0)
       (effects (font (size 1.27 1.27)) (justify left))
     )
@@
   (symbol (lib_id "Device:R_Small_US") (at 100.965 35.56 90) (unit 1)
     (in_bom yes) (on_board yes)
-    (property "Reference" "R?" (id 0) (at 99.06 36.83 90)
+    (property "Reference" "R34" (id 0) (at 99.06 36.83 90)
       (effects (font (size 1.27 1.27)) (justify left))
     )
@@
   (symbol (lib_id "power:GNDREF") (at 110.49 77.47 0) (unit 1)
     (in_bom yes) (on_board yes) (fields_autoplaced)
-    (property "Reference" "#PWR?" (id 0) (at 110.49 83.82 0)
+    (property "Reference" "#PWR068" (id 0) (at 110.49 83.82 0)
       (effects (font (size 1.27 1.27)) hide)
     )
@@
   (symbol (lib_id "Device:R_Small_US") (at 110.49 69.85 180) (unit 1)
     (in_bom yes) (on_board yes)
-    (property "Reference" "R?" (id 0) (at 112.395 71.755 90))
+    (property "Reference" "R37" (id 0) (at 112.395 71.755 90))
     (property "Value" "1K" (id 1) (at 112.395 67.31 90))
     (property "Footprint" "Resistor_SMD:R_0805_2012Metric" (id 2) (at 110.49 69.85 0)
@@
   (symbol (lib_id "power:GNDREF") (at 36.83 33.02 270) (unit 1)
     (in_bom yes) (on_board yes)
-    (property "Reference" "#PWR?" (id 0) (at 30.48 33.02 0)
+    (property "Reference" "#PWR063" (id 0) (at 30.48 33.02 0)
       (effects (font (size 1.27 1.27)) hide)
     )
@@
   (symbol (lib_id "Device:R_Small_US") (at 39.37 46.99 180) (unit 1)
     (in_bom yes) (on_board yes)
-    (property "Reference" "R?" (id 0) (at 36.195 46.99 90))
+    (property "Reference" "R30" (id 0) (at 36.195 46.99 90))
     (property "Value" "0R_NM" (id 1) (at 41.91 46.99 90))
     (property "Footprint" "Resistor_SMD:R_0805_2012Metric" (id 2) (at 39.37 46.99 0)
