File: ramps.kicad_sch (KiCad schematic)
At the start: 54 parts, among them J10 X, J11 E, J12 YM, J13 Y, J14 ZM, J15 Z, J16 Z, J3 X-, J4 Thermistor, J5 Y-, J6 Z-, J7 Heaters & Fans, J8 XM, J9 EM, Q1 Mos, Q2 Mos, Q3 Mos

Commit message: hebele
Parts:
- removed C20: 100uF, Capacitor_SMD:C_0805_2012Metric, symbol Device:C_Small
- removed J12: YM, Connector_PinHeader_2.54mm:PinHeader_2x03_P2.54mm_Vertical, symbol Connector_Generic:Conn_02x03_Odd_Even
- removed J14: ZM, Connector_PinHeader_2.54mm:PinHeader_2x03_P2.54mm_Vertical, symbol Connector_Generic:Conn_02x03_Odd_Even
- removed J8: XM, Connector_PinHeader_2.54mm:PinHeader_2x03_P2.54mm_Vertical, symbol Connector_Generic:Conn_02x03_Odd_Even
- removed J9: EM, Connector_PinHeader_2.54mm:PinHeader_2x03_P2.54mm_Vertical, symbol Connector_Generic:Conn_02x03_Odd_Even
- C16, C17, C18, C19: footprint Capacitor_SMD:C_0805_2012Metric -> Capacitor_SMD:CP_Elec_6.3x7.7
- J7: footprint Connector_Phoenix_MSTB:PhoenixContact_MSTBVA_2,5_6-G-5,08_1x06_P5.08mm_Vertical -> TerminalBlock_Phoenix:TerminalBlock_Phoenix_MKDS-1,5-6-5.08_1x06_P5.08mm_Horizontal
- Q1, Q2, Q3: footprint (none) -> Package_TO_SOT_SMD:TO-263-2
Connections:
- net ME1 is gone; now on net ME0: A2.11 (M1)
- net ME2 is gone; now on net ME0: A2.12 (M2)
- net MX0 is gone; now on net ME0: A1.10 (M0), R26.1
- net MX1 is gone; now on net ME0: A1.11 (M1)
- net MX2 is gone; now on net ME0: A1.12 (M2)
- net MY0 is gone; now on net ME0: A3.10 (M0), R29.1
- net MY1 is gone; now on net ME0: A3.11 (M1)
- net MY2 is gone; now on net ME0: A3.12 (M2)
- net MZ0 is gone; now on net ME0: A4.10 (M0), R31.1
- net MZ1 is gone; now on net ME0: A4.11 (M1)
- net MZ2 is gone; now on net ME0: A4.12 (M2)
- net VCC is gone; now on net ME0: J3.3 (Pin_3), J5.3 (Pin_3), J6.3 (Pin_3), R11.2, R18.2, R22.2, R24.2, R25.2, R28.2, R30.2

Commit message: Schematic_ok
Parts:
- removed A1, A2, A3, A4: Pololu_Breakout_DRV8825, Module:Pololu_Breakout-16_15.2x20.3mm, symbol Driver_Motor:Pololu_Breakout_DRV8825
- removed J10: X, Connector_PinHeader_2.54mm:PinHeader_1x04_P2.54mm_Vertical, symbol Connector_Generic:Conn_01x04
- removed J11: E, Connector_PinHeader_2.54mm:PinHeader_1x04_P2.54mm_Vertical, symbol Connector_Generic:Conn_01x04
- removed J13: Y, Connector_PinHeader_2.54mm:PinHeader_1x04_P2.54mm_Vertical, symbol Connector_Generic:Conn_01x04
- removed J15, J16: Z, Connector_PinHeader_2.54mm:PinHeader_1x04_P2.54mm_Vertical, symbol Connector_Generic:Conn_01x04
- removed J3: X-, Connector_PinHeader_2.54mm:PinHeader_1x03_P2.54mm_Vertical, symbol Connector_Generic:Conn_01x03
- removed J5: Y-, Connector_PinHeader_2.54mm:PinHeader_1x03_P2.54mm_Vertical, symbol Connector_Generic:Conn_01x03
- removed J6: Z-, Connector_PinHeader_2.54mm:PinHeader_1x03_P2.54mm_Vertical, symbol Connector_Generic:Conn_01x03
- removed R24, R25, R28, R30: 10K, Resistor_SMD:R_0805_2012Metric, symbol Device:R_Small_US
- removed R26, R27, R29, R31: 100K, Resistor_SMD:R_0805_2012Metric, symbol Device:R_Small_US
- added A? (x4): DRIVER, Module:Pololu_Breakout-16_15.2x20.3mm, symbol Driver_Motor:Pololu_Breakout_A4988
- added C20: 100uF, Capacitor_SMD:C_0805_2012Metric, symbol Device:C_Small
- added C? (x4): 100uF 35V, Capacitor_SMD:CP_Elec_6.3x7.7, symbol Device:C_Polarized_Small
- added J?: X_END, TerminalBlock_MetzConnect:TerminalBlock_MetzConnect_Type086_RT03406HBLC_1x06_P3.81mm_Horizontal, symbol Connector_Generic:Conn_01x06
- added J? (x4): Conn_01x04, TerminalBlock_MetzConnect:TerminalBlock_MetzConnect_Type086_RT03404HBLC_1x04_P3.81mm_Horizontal, symbol Connector_Generic:Conn_01x04
- added J? (x4): MCU_PROG, Connector_PinHeader_2.54mm:PinHeader_2x03_P2.54mm_Vertical, symbol Connector_Generic:Conn_02x03_Odd_Even
- added J?: Y_END, TerminalBlock_MetzConnect:TerminalBlock_MetzConnect_Type086_RT03406HBLC_1x06_P3.81mm_Horizontal, symbol Connector_Generic:Conn_01x06
- added J?: Z_END, TerminalBlock_MetzConnect:TerminalBlock_MetzConnect_Type086_RT03406HBLC_1x06_P3.81mm_Horizontal, symbol Connector_Generic:Conn_01x06
- added R? (x4): 100K, Resistor_SMD:R_0805_2012Metric, symbol Device:R_Small_US
- added R? (x4): 10K, Resistor_SMD:R_0805_2012Metric, symbol Device:R_Small_US
- C13, C14, C15: footprint Capacitor_SMD:C_0805_2012Metric -> Capacitor_SMD:CP_Elec_4x5.7
- C16, C17, C18, C19: footprint Capacitor_SMD:CP_Elec_6.3x7.7 -> Capacitor_SMD:C_0805_2012Metric
- J4: footprint Connector_PinHeader_2.54mm:PinHeader_1x06_P2.54mm_Vertical -> TerminalBlock_MetzConnect:TerminalBlock_MetzConnect_Type086_RT03406HBLC_1x06_P3.81mm_Horizontal
- J7: footprint TerminalBlock_Phoenix:TerminalBlock_Phoenix_MKDS-1,5-6-5.08_1x06_P5.08mm_Horizontal -> Connector_Phoenix_MC:PhoenixContact_MC_1,5_6-G-3.81_1x06_P3.81mm_Horizontal
- Q1, Q2, Q3: footprint Package_TO_SOT_SMD:TO-263-2 -> Package_TO_SOT_SMD:TO-263-5_TabPin3
Connections:
- net GND: no longer C13.2, C14.2, C15.2, C16.2, C17.2, C18.2, C19.2, J4.1 (Pin_1), J4.3 (Pin_3), J4.5 (Pin_5), Q1.2 (S), Q2.2 (S), Q3.2 (S), R15.2, R16.2, R17.2
- net 12V renamed +12V
- net +12V: now also A?.8 (VMOT), A?.8 (VMOT), A?.8 (VMOT), A?.8 (VMOT), C20.1, C?.1, C?.1, C?.1, C?.1
- net ME0 renamed VCC
- new net: A?.13 (~{RESET}), A?.14 (~{SLEEP}) (x4)
- new net: A?.3 (1B), J?.1 (Pin_1) (x4)
- new net: A?.4 (1A), J?.2 (Pin_2) (x4)
- new net: A?.5 (2A), J?.3 (Pin_3) (x4)
- new net: A?.6 (2B), J?.4 (Pin_4) (x4)
- new net +5V: A?.2 (VDD), A?.2 (VDD), A?.2 (VDD), A?.2 (VDD), J?.2 (Pin_2), J?.2 (Pin_2), J?.2 (Pin_2), J?.2 (Pin_2), J?.3 (Pin_3), J?.3 (Pin_3), J?.3 (Pin_3), J?.4 (Pin_4), J?.4 (Pin_4), J?.4 (Pin_4), J?.4 (Pin_4), J?.6 (Pin_6), J?.6 (Pin_6), J?.6 (Pin_6), J?.6 (Pin_6), J?.6 (Pin_6), J?.6 (Pin_6), R?.1, R?.1, R?.1, R?.1
- new net EMS1: A?.10 (MS1), J?.1 (Pin_1), R?.2
- new net EMS2: A?.11 (MS2), J?.3 (Pin_3)
- new net EMS3: A?.12 (MS3), J?.5 (Pin_5)
- new net E_DIR: A?.16 (DIR)
- new net E_EN: A?.9 (~{ENABLE}), R?.2
- new net E_STEP: A?.15 (STEP)
- new net GNDREF: A?.1 (GND), A?.1 (GND), A?.1 (GND), A?.1 (GND), A?.7 (GND), A?.7 (GND), A?.7 (GND), A?.7 (GND), C13.2, C14.2, C15.2, C16.2, C17.2, C18.2, C19.2, C20.2, C?.2, C?.2, C?.2, C?.2, J4.1 (Pin_1), J4.3 (Pin_3), J4.5 (Pin_5), J?.2 (Pin_2), J?.2 (Pin_2), J?.2 (Pin_2), J?.5 (Pin_5), J?.5 (Pin_5), J?.5 (Pin_5), Q1.2 (S), Q2.2 (S), Q3.2 (S), R15.2, R16.2, R17.2, R?.1, R?.1, R?.1, R?.1
- new net XMS1: A?.10 (MS1), J?.1 (Pin_1), R?.2
- new net XMS2: A?.11 (MS2), J?.3 (Pin_3)
- new net XMS3: A?.12 (MS3), J?.5 (Pin_5)
- new net X_DIR: A?.16 (DIR)
- new net X_EN: A?.9 (~{ENABLE}), R?.2
- new net X_MAX: J?.4 (Pin_4)
- new net X_MIN: J?.1 (Pin_1)
- new net X_STEP: A?.15 (STEP)
- new net YMS1: A?.10 (MS1), J?.1 (Pin_1), R?.2
- new net YMS2: A?.11 (MS2), J?.3 (Pin_3)
- new net YMS3: A?.12 (MS3), J?.5 (Pin_5)
- new net Y_DIR: A?.16 (DIR)
- new net Y_EN: A?.9 (~{ENABLE}), R?.2
- new net Y_MAX: J?.4 (Pin_4)
- new net Y_MIN: J?.1 (Pin_1)
- new net Y_STEP: A?.15 (STEP)
- new net ZMS1: A?.10 (MS1), J?.1 (Pin_1), R?.2
- new net ZMS2: A?.11 (MS2), J?.3 (Pin_3)
- new net ZMS3: A?.12 (MS3), J?.5 (Pin_5)
- new net Z_DIR: A?.16 (DIR)
- new net Z_EN: A?.9 (~{ENABLE}), R?.2
- new net Z_MAX: J?.4 (Pin_4)
- new net Z_MIN: J?.1 (Pin_1)
- new net Z_STEP: A?.15 (STEP)
- no-connect marks 4 -> 0
Other:
- note added: "EXTRUDER"
- note added: "XSTEP"
- note added: "YSTEP"
- note added: "ZSTEP"
- note removed: "Stepper Drivers"
- moved on the sheet: C13, C14, C15, C16, C17, C18, C19, D8, J4, R11, R18, R22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

Commit message: PCB
Parts:
- removed D8: LED, LED_SMD:LED_0805_2012Metric, symbol Device:LED_Small
- removed R23: 1K, Resistor_SMD:R_0805_2012Metric, symbol Device:R_Small_US
- added R39, R40, R41, R42, R43, R44: 4K7, Resistor_SMD:R_0805_2012Metric_Pad1.20x1.40mm_HandSolder, symbol Device:R_Small_US
- J11, J13, J15, J9: renamed from J?; footprint TerminalBlock_MetzConnect:TerminalBlock_MetzConnect_Type086_RT03404HBLC_1x04_P3.81mm_Horizontal -> Connector_Phoenix_MC:PhoenixContact_MC_1,5_4-G-3.81_1x04_P3.81mm_Horizontal
- J8: renamed from J7; footprint Connector_Phoenix_MC:PhoenixContact_MC_1,5_6-G-3.81_1x06_P3.81mm_Horizontal -> TerminalBlock_Phoenix:TerminalBlock_Phoenix_MKDS-1,5-6_1x06_P5.00mm_Horizontal
- Q1, Q2, Q3: footprint Package_TO_SOT_SMD:TO-263-5_TabPin3 -> Package_TO_SOT_SMD:TO-263-2
- gave numbers to parts that had none: 23
- renumbered C14 to C10, C15 to C11, C13 to C9, D5 to D6, D6 to D7, D7 to D8, J4 to J5, R12 to R10, R13 to R11, R14 to R12, R15 to R13, R16 to R14, R17 to R15, R18 to R16, R19 to R17, R20 to R18, R21 to R19, R22 to R20, R11 to R9
Connections:
- net +5V: now also J7.6 (Pin_6), R39.1, R40.1, R41.1, R42.1, R43.1, R44.1
- net X_MAX: now also R40.2
- net X_MIN: now also R39.2
- net Y_MAX: now also R42.2
- net Y_MIN: now also R41.2
- net Z_MAX: now also R44.2
- net Z_MIN: now also R43.2
Other:
- note removed: "LED"
- moved on the sheet: J4, J6, J7

Commit message: finish
Parts:
- R39, R40, R41, R42, R43, R44: footprint Resistor_SMD:R_0805_2012Metric_Pad1.20x1.40mm_HandSolder -> Resistor_SMD:R_0805_2012Metric
Connections:
- net VCC is gone; now on net +5V: R16.2, R20.2, R9.2
- net THERM0: now also C11.1, J5.6 (Pin_6), R20.1; no longer C9.1, J5.2 (Pin_2), R9.1
- net THERM2: now also C9.1, J5.2 (Pin_2), R9.1; no longer C11.1, J5.6 (Pin_6), R20.1
Changed lines of the file:
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@@
+    (stroke (width 0) (type default) (color 0 0 0 0))
+  )
+  (wire (pts (xy 36.83 92.075) (xy 36.83 92.71))
     (stroke (width 0) (type default) (color 0 0 0 0))
   )
@@
   )
   (wire (pts (xy 107.315 33.02) (xy 105.41 33.02))
+    (stroke (width 0) (type default) (color 0 0 0 0))
+  )
+  (wire (pts (xy 36.83 92.71) (xy 38.1 92.71))
     (stroke (width 0) (type default) (color 0 0 0 0))
   )
@@
     )
   )
-  (global_label "THERM2" (shape input) (at 60.96 100.33 270) (fields_autoplaced)
-    (effects (font (size 1.27 1.27)) (justify right))
-    (property "Intersheet References" "${INTERSHEET_REFS}" (id 0) (at 60.8806 110.1212 90)
+  (global_label "THERM2" (shape input) (at 27.94 100.33 270) (fields_autoplaced)
+    (effects (font (size 1.27 1.27)) (justify right))
+    (property "Intersheet References" "${INTERSHEET_REFS}" (id 0) (at 27.8606 110.1212 90)
       (effects (font (size 1.27 1.27)) (justify right) hide)
     )
@@
     (effects (font (size 1.27 1.27)) (justify right))
     (property "Intersheet References" "${INTERSHEET_REFS}" (id 0) (at 97.9169 55.8006 0)
-      (effects (font (size 1.27 1.27)) (justify right) hide)
-    )
-  )
-  (global_label "VCC" (shape input) (at 38.1 92.71 180) (fields_autoplaced)
-    (effects (font (size 1.27 1.27)) (justify right))
-    (property "Intersheet References" "${INTERSHEET_REFS}" (id 0) (at 32.0583 92.6306 0)
       (effects (font (size 1.27 1.27)) (justify right) hide)
     )
@@
     )
   )
-  (global_label "THERM0" (shape input) (at 27.94 100.33 270) (fields_autoplaced)
-    (effects (font (size 1.27 1.27)) (justify right))
-    (property "Intersheet References" "${INTERSHEET_REFS}" (id 0) (at 27.8606 110.1212 90)
+  (global_label "THERM0" (shape input) (at 60.96 100.33 270) (fields_autoplaced)
+    (effects (font (size 1.27 1.27)) (justify right))
+    (property "Intersheet References" "${INTERSHEET_REFS}" (id 0) (at 60.8806 110.1212 90)
       (effects (font (size 1.27 1.27)) (justify right) hide)
     )
@@
     )
   )
-  (global_label "VCC" (shape input) (at 54.61 92.71 180) (fields_autoplaced)
-    (effects (font (size 1.27 1.27)) (justify right))
-    (property "Intersheet References" "${INTERSHEET_REFS}" (id 0) (at 48.5683 92.6306 0)
-      (effects (font (size 1.27 1.27)) (justify right) hide)
-    )
-  )
-  (global_label "VCC" (shape input) (at 21.59 92.71 180) (fields_autoplaced)
-    (effects (font (size 1.27 1.27)) (justify right))
-    (property "Intersheet References" "${INTERSHEET_REFS}" (id 0) (at 15.5483 92.6306 0)
-      (effects (font (size 1.27 1.27)) (justify right) hide)
-    )
-  )
   (global_label "ZMS3" (shape input) (at 271.145 67.945 180) (fields_autoplaced)
     (effects (font (size 1.27 1.27)) (justify right))
@@
     (property "Reference" "R39" (id 0) (at 27.94 131.445 90))
     (property "Value" "4K7" (id 1) (at 27.94 127 90))
-    (property "Footprint" "Resistor_SMD:R_0805_2012Metric_Pad1.20x1.40mm_HandSolder" (id 2) (at 27.94 129.54 0)
+    (property "Footprint" "Resistor_SMD:R_0805_2012Metric" (id 2) (at 27.94 129.54 0)
       (effects (font (size 1.27 1.27)) hide)
     )
@@
     (pin "2")
   )
+  (symbol (lib_id "power:+5V") (at 54.61 92.71 0) (unit 1)
+    (in_bom yes) (on_board yes)
+    (property "Reference" "#PWR0105" (id 0) (at 54.61 96.52 0)
+      (effects (font (size 1.27 1.27)) hide)
+    )
+    (property "Value" "+5V" (id 1) (at 53.34 92.71 0)
+      (effects (font (size 1.27 1.27)) (justify right))
+    )
+    (property "Footprint" "" (id 2) (at 54.61 92.71 0)
+      (effects (font (size 1.27 1.27)) hide)
+    )
+    (property "Datasheet" "" (id 3) (at 54.61 92.71 0)
+      (effects (font (size 1.27 1.27)) hide)
+    )
+    (pin "1")
+  )
   (symbol (lib_id "Device:R_Small_US") (at 58.42 129.573 270) (unit 1)
     (in_bom yes) (on_board yes)
     (property "Reference" "R42" (id 0) (at 58.42 131.478 90))
     (property "Value" "4K7" (id 1) (at 58.42 127.033 90))
-    (property "Footprint" "Resistor_SMD:R_0805_2012Metric_Pad1.20x1.40mm_HandSolder" (id 2) (at 58.42 129.573 0)
+    (property "Footprint" "Resistor_SMD:R_0805_2012Metric" (id 2) (at 58.42 129.573 0)
       (effects (font (size 1.27 1.27)) hide)
     )
@@
     (pin "1")
     (pin "2")
+  )
+  (symbol (lib_id "power:+5V") (at 36.83 92.075 0) (unit 1)
+    (in_bom yes) (on_board yes)
+    (property "Reference" "#PWR0106" (id 0) (at 36.83 95.885 0)
+      (effects (font (size 1.27 1.27)) hide)
+    )
+    (property "Value" "+5V" (id 1) (at 36.195 92.075 0)
+      (effects (font (size 1.27 1.27)) (justify right))
+    )
+    (property "Footprint" "" (id 2) (at 36.83 92.075 0)
+      (effects (font (size 1.27 1.27)) hide)
+    )
+    (property "Datasheet" "" (id 3) (at 36.83 92.075 0)
+      (effects (font (size 1.27 1.27)) hide)
+    )
+    (pin "1")
   )
   (symbol (lib_id "power:GNDREF") (at 81.28 135.89 0) (unit 1)
@@
     (property "Reference" "R43" (id 0) (at 73.66 131.445 90))
     (property "Value" "4K7" (id 1) (at 73.66 127 90))
-    (property "Footprint" "Resistor_SMD:R_0805_2012Metric_Pad1.20x1.40mm_HandSolder" (id 2) (at 73.66 129.54 0)
+    (property "Footprint" "Resistor_SMD:R_0805_2012Metric" (id 2) (at 73.66 129.54 0)
       (effects (font (size 1.27 1.27)) hide)
     )
@@
     (property "Reference" "R41" (id 0) (at 50.8 131.445 90))
     (property "Value" "4K7" (id 1) (at 50.8 127 90))
-    (property "Footprint" "Resistor_SMD:R_0805_2012Metric_Pad1.20x1.40mm_HandSolder" (id 2) (at 50.8 129.54 0)
+    (property "Footprint" "Resistor_SMD:R_0805_2012Metric" (id 2) (at 50.8 129.54 0)
       (effects (font (size 1.27 1.27)) hide)
     )
@@
     (property "Reference" "R40" (id 0) (at 35.56 131.5209 90))
     (property "Value" "4K7" (id 1) (at 35.56 127.0759 90))
-    (property "Footprint" "Resistor_SMD:R_0805_2012Metric_Pad1.20x1.40mm_HandSolder" (id 2) (at 35.56 129.6159 0)
+    (property "Footprint" "Resistor_SMD:R_0805_2012Metric" (id 2) (at 35.56 129.6159 0)
       (effects (font (size 1.27 1.27)) hide)
     )
@@
     )
     (property "Datasheet" "" (id 3) (at 304.165 29.845 0)
+      (effects (font (size 1.27 1.27)) hide)
+    )
+    (pin "1")
+  )
+  (symbol (lib_id "power:+5V") (at 21.59 92.71 0) (unit 1)
+    (in_bom yes) (on_board yes)
+    (property "Reference" "#PWR0107" (id 0) (at 21.59 96.52 0)
+      (effects (font (size 1.27 1.27)) hide)
+    )
+    (property "Value" "+5V" (id 1) (at 20.32 92.71 0)
+      (effects (font (size 1.27 1.27)) (justify right))
+    )
+    (property "Footprint" "" (id 2) (at 21.59 92.71 0)
+      (effects (font (size 1.27 1.27)) hide)
+    )
+    (property "Datasheet" "" (id 3) (at 21.59 92.71 0)
       (effects (font (size 1.27 1.27)) hide)
     )
@@
     (property "Reference" "R44" (id 0) (at 81.28 131.445 90))
     (property "Value" "4K7" (id 1) (at 81.28 127 90))
-    (property "Footprint" "Resistor_SMD:R_0805_2012Metric_Pad1.20x1.40mm_HandSolder" (id 2) (at 81.28 129.54 0)
-      (effects (font (size 1.27 1.27)) hide)
-    )
+    (property "Footprint" "Resistor_SMD:R_0805_2012Metric" (id 2) (at 81.28 129.54 0)
+      (effects (font (size 1.27 1.27)) hide)
+    )
