File: 3dprinter.kicad_sch (KiCad schematic)
At the start: 35 parts, among them J1 6P IDC CONNECTOR, J17 Conn_01x02, J2 USB_B, SW1 SW_Push, U1 ATmega2560-16A, U2 CH340G, U3 LM78M05_TO252, Y1 16MHZ, Y2 12MHZ

Commit message: hebele
Parts:
- C12: footprint Capacitor_SMD:C_0805_2012Metric -> Capacitor_SMD:CP_Elec_6.3x7.7
- J1: footprint Connector_PinHeader_1.00mm:PinHeader_2x03_P1.00mm_Vertical -> Connector_PinHeader_2.54mm:PinHeader_2x03_P2.54mm_Vertical
- J17: footprint Connector_Phoenix_MSTB:PhoenixContact_MSTBVA_2,5_2-G-5,08_1x02_P5.08mm_Vertical -> TerminalBlock_Phoenix:TerminalBlock_Phoenix_MKDS-1,5-2-5.08_1x02_P5.08mm_Horizontal
Connections:
- net PB1(SCK) is gone; now on net SCK: J1.3 (Pin_3)
- net PB2(MOSI) is gone; now on net MOSI: J1.4 (Pin_4)
- net PB3(MISO) is gone; now on net MISO: J1.1 (Pin_1)
- net PB7: now also U1.26 (PB7)
- no-connect marks 41 -> 40
Changed lines of the file:
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@@
   (no_connect (at 71.12 129.54))
   (no_connect (at 71.12 139.7))
-  (no_connect (at 71.12 76.2))
   (no_connect (at 71.12 132.08))
   (no_connect (at 262.89 48.26))
@@
     (stroke (width 0) (type default) (color 0 0 0 0))
   )
+  (wire (pts (xy 71.12 76.2) (xy 73.66 76.2))
+    (stroke (width 0) (type default) (color 0 0 0 0))
+  )
   (wire (pts (xy 71.12 60.96) (xy 72.39 60.96))
     (stroke (width 0) (type default) (color 0 0 0 0))
@@
     )
   )
-  (global_label "PB2(MOSI)" (shape input) (at 121.92 48.26 0) (fields_autoplaced)
-    (effects (font (size 1.27 1.27)) (justify left))
-    (property "Intersheet References" "${INTERSHEET_REFS}" (id 0) (at 134.3721 48.1806 0)
-      (effects (font (size 1.27 1.27)) (justify left) hide)
-    )
-  )
-  (global_label "PB3(MISO)" (shape input) (at 106.68 45.72 180) (fields_autoplaced)
-    (effects (font (size 1.27 1.27)) (justify right))
-    (property "Intersheet References" "${INTERSHEET_REFS}" (id 0) (at 94.2279 45.7994 0)
+  (global_label "MOSI" (shape input) (at 121.92 48.26 0) (fields_autoplaced)
+    (effects (font (size 1.27 1.27)) (justify left))
+    (property "Intersheet References" "${INTERSHEET_REFS}" (id 0) (at 128.9293 48.1806 0)
+      (effects (font (size 1.27 1.27)) (justify left) hide)
+    )
+  )
+  (global_label "MISO" (shape input) (at 106.68 45.72 180) (fields_autoplaced)
+    (effects (font (size 1.27 1.27)) (justify right))
+    (property "Intersheet References" "${INTERSHEET_REFS}" (id 0) (at 99.6707 45.6406 0)
       (effects (font (size 1.27 1.27)) (justify right) hide)
     )
@@
     )
   )
-  (global_label "PB1(SCK)" (shape input) (at 106.68 48.26 180) (fields_autoplaced)
-    (effects (font (size 1.27 1.27)) (justify right))
-    (property "Intersheet References" "${INTERSHEET_REFS}" (id 0) (at 95.0745 48.3394 0)
+  (global_label "SCK" (shape input) (at 106.68 48.26 180) (fields_autoplaced)
+    (effects (font (size 1.27 1.27)) (justify right))
+    (property "Intersheet References" "${INTERSHEET_REFS}" (id 0) (at 100.5174 48.1806 0)
       (effects (font (size 1.27 1.27)) (justify right) hide)
     )
@@
     (property "Intersheet References" "${INTERSHEET_REFS}" (id 0) (at 98.5217 50.7206 0)
       (effects (font (size 1.27 1.27)) (justify right) hide)
+    )
+  )
+  (global_label "PB7" (shape input) (at 73.66 76.2 0) (fields_autoplaced)
+    (effects (font (size 1.27 1.27)) (justify left))
+    (property "Intersheet References" "${INTERSHEET_REFS}" (id 0) (at 79.8226 76.1206 0)
+      (effects (font (size 1.27 1.27)) (justify left) hide)
     )
   )
@@
     (property "Reference" "J1" (id 0) (at 114.3 39.37 0))
     (property "Value" "6P IDC CONNECTOR" (id 1) (at 114.3 41.91 0))
-    (property "Footprint" "Connector_PinHeader_1.00mm:PinHeader_2x03_P1.00mm_Vertical" (id 2) (at 113.03 48.26 0)
+    (property "Footprint" "Connector_PinHeader_2.54mm:PinHeader_2x03_P2.54mm_Vertical" (id 2) (at 113.03 48.26 0)
       (effects (font (size 1.27 1.27)) hide)
     )
@@
     (property "Reference" "C12" (id 0) (at 201.93 39.37 90))
     (property "Value" "22uF 25V SMD" (id 1) (at 201.93 41.91 90))
-    (property "Footprint" "Capacitor_SMD:C_0805_2012Metric" (id 2) (at 201.93 44.45 0)
+    (property "Footprint" "Capacitor_SMD:CP_Elec_6.3x7.7" (id 2) (at 201.93 44.45 0)
       (effects (font (size 1.27 1.27)) hide)
     )
@@
       (effects (font (size 1.27 1.27)) (justify left))
     )
-    (property "Footprint" "Connector_Phoenix_MSTB:PhoenixContact_MSTBVA_2,5_2-G-5,08_1x02_P5.08mm_Vertical" (id 2) (at 146.05 69.85 0)
+    (property "Footprint" "TerminalBlock_Phoenix:TerminalBlock_Phoenix_MKDS-1,5-2-5.08_1x02_P5.08mm_Horizontal" (id 2) (at 146.05 69.85 0)
       (effects (font (size 1.27 1.27)) hide)
     )
@@
     )
     (path "/b4aa4a0b-de28-4387-a0ea-9b131fef418f"
-      (reference "C12") (unit 1) (value "22uF 25V SMD") (footprint "Capacitor_SMD:C_0805_2012Metric")
+      (reference "C12") (unit 1) (value "22uF 25V SMD") (footprint "Capacitor_SMD:CP_Elec_6.3x7.7")
     )
     (path "/a38a02bc-82b4-4ed0-acec-d0a59f3ca71c/93cf6b4e-cd7b-4f85-9cca-dec9452ee825"
@@
     )
     (path "/a38a02bc-82b4-4ed0-acec-d0a59f3ca71c/34093c9c-d95f-447c-8a26-5c4272f75992"
-      (reference "C16") (unit 1) (value "100uF") (footprint "Capacitor_SMD:C_0805_2012Metric")
+      (reference "C16") (unit 1) (value "100uF") (footprint "Capacitor_SMD:CP_Elec_6.3x7.7")
     )
     (path "/a38a02bc-82b4-4ed0-acec-d0a59f3ca71c/12c3d759-8e3b-4487-82bf-62315962caf7"
-      (reference "C17") (unit 1) (value "100uF") (footprint "Capacitor_SMD:C_0805_2012Metric")
+      (reference "C17") (unit 1) (value "100uF") (footprint "Capacitor_SMD:CP_Elec_6.3x7.7")
     )
     (path "/a38a02bc-82b4-4ed0-acec-d0a59f3ca71c/98de819c-394a-41f8-8f5d-1f9dfc4db40e"
-      (reference "C18") (unit 1) (value "100uF") (footprint "Capacitor_SMD:C_0805_2012Metric")
+      (reference "C18") (unit 1) (value "100uF") (footprint "Capacitor_SMD:CP_Elec_6.3x7.7")
     )
     (path "/a38a02bc-82b4-4ed0-acec-d0a59f3ca71c/c4a9c044-9cc2-4f80-a0d8-f23fa8ca900c"
-      (reference "C19") (unit 1) (value "100uF") (footprint "Capacitor_SMD:C_0805_2012Metric")
-    )
-    (path "/a38a02bc-82b4-4ed0-acec-d0a59f3ca71c/3d1bfd9a-7401-4993-9181-54015b650bc4"
-      (reference "C20") (unit 1) (value "100uF") (footprint "Capacitor_SMD:C_0805_2012Metric")
+      (reference "C19") (unit 1) (value "100uF") (footprint "Capacitor_SMD:CP_Elec_6.3x7.7")
     )
     (path "/17afffa6-f020-49f2-b803-5d65f9891e60"
@@
     )
     (path "/88c272e3-7b52-4676-9687-514e2ed58139"
-      (reference "J1") (unit 1) (value "6P IDC CONNECTOR") (footprint "Connector_PinHeader_1.00mm:PinHeader_2x03_P1.00mm_Vertical")
+      (reference "J1") (unit 1) (value "6P IDC CONNECTOR") (footprint "Connector_PinHeader_2.54mm:PinHeader_2x03_P2.54mm_Vertical")
     )
     (path "/17f9818c-2665-471f-8cd4-f852a2eb8fe2"
@@
     )
     (path "/a38a02bc-82b4-4ed0-acec-d0a59f3ca71c/f8ff46ec-1e7a-47fa-8ba7-e09a1b20eb85"
-      (reference "J7") (unit 1) (value "Heaters & Fans") (footprint "Connector_Phoenix_MSTB:PhoenixContact_MSTBVA_2,5_6-G-5,08_1x06_P5.08mm_Vertical")
-    )
-    (path "/a38a02bc-82b4-4ed0-acec-d0a59f3ca71c/a5abc946-342c-4223-b8cb-ce56a6c42925"
-      (reference "J8") (unit 1) (value "XM") (footprint "Connector_PinHeader_2.54mm:PinHeader_2x03_P2.54mm_Vertical")
-    )
-    (path "/a38a02bc-82b4-4ed0-acec-d0a59f3ca71c/2cbc97f2-47e2-4587-828d-a18ae6121e21"
-      (reference "J9") (unit 1) (value "EM") (footprint "Connector_PinHeader_2.54mm:PinHeader_2x03_P2.54mm_Vertical")
+      (reference "J7") (unit 1) (value "Heaters & Fans") (footprint "TerminalBlock_Phoenix:TerminalBlock_Phoenix_MKDS-1,5-6-5.08_1x06_P5.08mm_Horizontal")
     )
     (path "/a38a02bc-82b4-4ed0-acec-d0a59f3ca71c/e9a3d620-6a6a-41df-b1b6-e72b93648522"
@@
       (reference "J11") (unit 1) (value "E") (footprint "Connector_PinHeader_2.54mm:PinHeader_1x04_P2.54mm_Vertical")
     )
-    (path "/a38a02bc-82b4-4ed0-acec-d0a59f3ca71c/11e2e07e-ca5d-4d79-90ac-f31339cca118"
-      (reference "J12") (unit 1) (value "YM") (footprint "Connector_PinHeader_2.54mm:PinHeader_2x03_P2.54mm_Vertical")
-    )
     (path "/a38a02bc-82b4-4ed0-acec-d0a59f3ca71c/9c5704f6-16fc-400b-9be9-7c5853185a6a"
       (reference "J13") (unit 1) (value "Y") (footprint "Connector_PinHeader_2.54mm:PinHeader_1x04_P2.54mm_Vertical")
     )
-    (path "/a38a02bc-82b4-4ed0-acec-d0a59f3ca71c/0f808b0c-2b8e-4b4a-b98f-bc65d5fa605e"
-      (reference "J14") (unit 1) (value "ZM") (footprint "Connector_PinHeader_2.54mm:PinHeader_2x03_P2.54mm_Vertical")
-    )
     (path "/a38a02bc-82b4-4ed0-acec-d0a59f3ca71c/0dd43b7c-8085-4d55-95f5-124c4518a304"
       (reference "J15") (unit 1) (value "Z") (footprint "Connector_PinHeader_2.54mm:PinHeader_1x04_P2.54mm_Vertical")
@@
     )
     (path "/e30b9aeb-cf7e-4b8f-8d7c-3c1c6f726652"
-      (reference "J17") (unit 1) (value "Conn_01x02") (footprint "Connector_Phoenix_MSTB:PhoenixContact_MSTBVA_2,5_2-G-5,08_1x02_P5.08mm_Vertical")
+      (reference "J17") (unit 1) (value "Conn_01x02") (footprint "TerminalBlock_Phoenix:TerminalBlock_Phoenix_MKDS-1,5-2-5.08_1x02_P5.08mm_Horizontal")
     )
     (path "/a38a02bc-82b4-4ed0-acec-d0a59f3ca71c/bd7afe7a-2382-4343-94f7-d3aeeeecee05"
-      (reference "Q1") (unit 1) (value "Mos") (footprint "")
+      (reference "Q1") (unit 1) (value "Mos") (footprint "Package_TO_SOT_SMD:TO-263-2")
     )
     (path "/a38a02bc-82b4-4ed0-acec-d0a59f3ca71c/86f579e5-b73e-454c-87c2-c84505a82bfe"
-      (reference "Q2") (unit 1) (value "Mos") (footprint "")
+      (reference "Q2") (unit 1) (value "Mos") (footprint "Package_TO_SOT_SMD:TO-263-2")
     )
     (path "/a38a02bc-82b4-4ed0-acec-d0a59f3ca71c/91e0766e-424c-4f56-9f8b-5f877424606a"
-      (reference "Q3") (unit 1) (value "Mos") (footprint "")
+      (reference "Q3") (unit 1) (value "Mos") (footprint "Package_TO_SOT_SMD:TO-263-2")
     )
     (path "/25909e86-1c5a-46f0-b549-a5bd102a2396"

Commit message: Schematic_ok
Parts:
- removed C1: 47uF, Capacitor_SMD:C_0805_2012Metric, symbol Device:C_Small
- removed C10, C11, C2, C3, C4, C5, C6, C7: 0.1uF, Capacitor_SMD:C_0805_2012Metric, symbol Device:C_Small
- removed C12: 22uF 25V SMD, Capacitor_SMD:CP_Elec_6.3x7.7, symbol Device:C_Polarized_Small_US
- removed C8, C9: 22pF, Capacitor_SMD:C_0805_2012Metric, symbol Device:C_Small
- removed D1, D2: LED, LED_SMD:LED_0805_2012Metric, symbol Device:LED_Small
- removed J2: USB_B, Connector_USB:USB_B_Lumberg_2411_02_Horizontal, symbol Connector:USB_B
- removed R10, R8, R9: 1K, Resistor_SMD:R_0805_2012Metric, symbol Device:R_Small_US
- removed R2, R4: 330, Resistor_SMD:R_0805_2012Metric, symbol Device:R_Small_US
- removed R3: 27R, Resistor_SMD:R_0805_2012Metric, symbol Device:R_Small_US
- removed R5: 1K, Resistor_SMD:R_0805_2012Metric_Pad1.20x1.40mm_HandSolder, symbol Device:R_Small_US
- removed SW1: SW_Push, Button_Switch_SMD:SW_Push_1P1T_NO_6x6mm_H9.5mm, symbol Switch:SW_Push
- removed U2: CH340G, Package_SO:SOIC-16_3.9x9.9mm_P1.27mm, symbol Interface_USB:CH340G
- removed U3: LM78M05_TO252, Package_TO_SOT_SMD:TO-252-2, symbol Regulator_Linear:LM78M05_TO252
- removed Y1: 16MHZ, Crystal:Crystal_SMD_HC49-SD, symbol Device:Resonator_Small
- removed Y2: 12MHZ, Crystal:Crystal_SMD_HC49-SD, symbol Device:Crystal_Small
- added C?: 47uF, Capacitor_SMD:C_0805_2012Metric_Pad1.18x1.45mm_HandSolder, symbol Device:C_Small
- added C? (x4): 100nF, Capacitor_SMD:C_0805_2012Metric_Pad1.18x1.45mm_HandSolder, symbol Device:C_Small
- added C?: 100nF, Capacitor_SMD:C_0805_2012Metric, symbol Device:C_Small
- added C? (x2): 22pF, Capacitor_SMD:C_0805_2012Metric_Pad1.18x1.45mm_HandSolder, symbol Device:C_Small
- added D? (x2): LED_RED, LED_SMD:LED_0805_2012Metric_Pad1.15x1.40mm_HandSolder, symbol Device:LED_Small
- added D?: LED_GREEN, LED_SMD:LED_0805_2012Metric_Pad1.15x1.40mm_HandSolder, symbol Device:LED_Small
- added FB?: FerriteBead_Small, Capacitor_SMD:C_1206_3216Metric, symbol Device:FerriteBead_Small
- added J?: USB_B_Micro, Connector_USB:USB_Micro-B_GCT_USB3076-30-A, symbol Connector:USB_B_Micro
- added R?: 10K, Resistor_SMD:R_0805_2012Metric_Pad1.20x1.40mm_HandSolder, symbol Device:R_Small_US
- added R? (x3): 330R, Resistor_SMD:R_0805_2012Metric_Pad1.20x1.40mm_HandSolder, symbol Device:R_Small_US
- added R?: 4K7, Resistor_SMD:R_0805_2012Metric, symbol Device:R_Small_US
- added SW?: 6x6 SMD, Button_Switch_SMD:SW_Push_1P1T_NO_6x6mm_H9.5mm, symbol Switch:SW_Push
- added Y?: 16MHz, Crystal:Crystal_SMD_HC49-SD, symbol Device:Crystal
- J1: footprint Connector_PinHeader_2.54mm:PinHeader_2x03_P2.54mm_Vertical -> Connector_PinHeader_1.00mm:PinHeader_2x03_P1.00mm_Vertical
- J17: footprint TerminalBlock_Phoenix:TerminalBlock_Phoenix_MKDS-1,5-2-5.08_1x02_P5.08mm_Horizontal -> Connector_Phoenix_MSTB:PhoenixContact_MSTBVA_2,5_2-G-5,08_1x02_P5.08mm_Vertical
Connections:
- net 5V is gone; now on net +5V: J1.2 (Pin_2), R6.1, U1.100 (AVCC)
- net D+: now also J?.3 (D+)
- net D-: now also J?.2 (D-)
- net GND: no longer J1.6 (Pin_6), J17.2 (Pin_2), U1.11 (GND), U1.32 (GND), U1.62 (GND), U1.81 (GND), U1.99 (GND)
- net PB7: no longer U1.26 (PB7)
- net XTAL1: now also C?.2, Y?.2
- net XTAL2: now also C?.2, Y?.1; no longer R1.1
- net GNDREF: now reaches R1.2
- net GNDREF: now also J1.6 (Pin_6), J17.2 (Pin_2), U1.11 (GND), U1.32 (GND), U1.62 (GND), U1.81 (GND), U1.99 (GND), C?.1, C?.1, C?.1, C?.1, C?.1, C?.2, J?.4 (ID), J?.5 (GND), J?.6 (Shield), R?.1, SW?.2
- net +5V: now reaches U1.10 (VCC), U1.31 (VCC), U1.61 (VCC), U1.80 (VCC)
- net +5V: now also C?.1, C?.2, C?.2, C?.2, C?.2, R?.1, R?.2, R?.2, R?.2
- net RXD: now reaches U1.2 (PE0)
- net RXD: now also D?.1 (K)
- net TXD: now reaches U1.3 (PE1)
- net TXD: now also D?.1 (K)
- net Z_MAX: now reaches U1.45 (PD2)
- net X_MAX: now reaches U1.6 (PE4)
- net Y_MAX: now reaches U1.63 (PJ0)
- net X_MIN: now reaches U1.7 (PE5)
- net 12V renamed +12V
- net AREF: no longer names the net of U1.98 (AREF)
- net AREF: now also C?.2
- net E0-EN renamed E_EN
- net EDIR renamed E_DIR
- net ESTEP renamed E_STEP
- net RESET renamed RES
- net RES: now also C?.1, R?.1, R?.2, SW?.1
- net X-EN renamed X_EN
- net XDIR renamed X_DIR
- net XSTEP renamed X_STEP
- net Y-EN renamed Y_EN
- net YDIR renamed Y_DIR
- net YMIN renamed Y_MIN
- net YSTEP renamed Y_STEP
- net Z-EN renamed Z_EN
- net ZDIR renamed Z_DIR
- net ZMIN renamed Z_MIN
- net ZSTEP renamed Z_STEP
- new net: D?.2 (A), R?.1 (x2)
- new net: C?.1, R1.1
- new net: D?.2 (A), U1.26 (PB7)
- new net: D?.1 (K), R?.2
- new net: FB?.1, J?.1 (VBUS)
- new net USB_VCC: FB?.2
- no-connect marks 40 -> 28
Other:
- added sheet FT232 (FT232.kicad_sch)
- added sheet POWER (POWER.kicad_sch)
- note added: "RESET"
- note added: "USB"
- note removed: "CH340"
- moved on the sheet: D3, D4, J1, J17, R1, R6, R7, U1

Commit message: PCB
Parts:
- removed D3, D4: LED, LED_SMD:LED_0805_2012Metric, symbol Device:LED_Small
- removed R6, R7: 1K, Resistor_SMD:R_0805_2012Metric, symbol Device:R_Small_US
- added H1, H2, H3, H4: MountingHole, MountingHole:MountingHole_3.2mm_M3_Pad_Via, symbol Mechanical:MountingHole
- J1: footprint Connector_PinHeader_1.00mm:PinHeader_2x03_P1.00mm_Vertical -> Connector_PinHeader_2.54mm:PinHeader_2x03_P2.54mm_Vertical
- J3: renamed from J17; footprint Connector_Phoenix_MSTB:PhoenixContact_MSTBVA_2,5_2-G-5,08_1x02_P5.08mm_Vertical -> TerminalBlock_Phoenix:TerminalBlock_Phoenix_MKDS-1,5-2-5.08_1x02_P5.08mm_Horizontal
- gave numbers to parts that had none: 20
- renumbered R1 to R3
Connections:
- net GNDREF: now also C6.1; no longer R3.2
- net XTAL1: now also R3.2
- net XTAL2: now also R3.1
Other:
- added sheet display (display.kicad_sch)
- moved on the sheet: C6, C7, R3

Commit message: finish
Parts:
- C1, C2, C3, C4, C5, C6, C7: footprint Capacitor_SMD:C_0805_2012Metric_Pad1.18x1.45mm_HandSolder -> Capacitor_SMD:C_0805_2012Metric
- D1, D2, D3: footprint LED_SMD:LED_0805_2012Metric_Pad1.15x1.40mm_HandSolder -> LED_SMD:LED_0805_2012Metric
- R1, R2, R4, R5: footprint Resistor_SMD:R_0805_2012Metric_Pad1.20x1.40mm_HandSolder -> Resistor_SMD:R_0805_2012Metric
Connections:
- net +5V: now also J1.4 (Pin_4); no longer J1.2 (Pin_2)
- net MOSI: now also J1.3 (Pin_3); no longer J1.4 (Pin_4)
- net RES: now also J1.2 (Pin_2); no longer J1.5 (Pin_5)
- net SCK: now also J1.5 (Pin_5); no longer J1.3 (Pin_3)
- net D8: now reaches U1.17 (PH5)
- net D9: now reaches U1.18 (PH6)
- net D10: now reaches U1.23 (PB4)
- net A10: no longer names the net of U1.87 (PK2)
- net A11: no longer names the net of U1.86 (PK3)
- net A12: no longer names the net of U1.85 (PK4)
- net A3: no longer names the net of U1.94 (PF3)
- net A4: no longer names the net of U1.93 (PF4)
- net A5: no longer names the net of U1.92 (PF5)
- net A9: no longer names the net of U1.88 (PK1)
- net D22: no longer names the net of U1.78 (PA0)
- net D40: no longer names the net of U1.52 (PG1)
- net D42: no longer names the net of U1.42 (PL7)
- net D44: no longer names the net of U1.40 (PL5)
- net SCL: no longer names the net of U1.43 (PD0)
- net SDA: no longer names the net of U1.44 (PD1)
- no-connect marks 28 -> 38

Commit message: comm
Changed lines of the file:
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@@
       (effects (font (size 1.27 1.27)) hide)
     )
-    (property "Value" "GNDREF" (id 1) (at 163.195 33.02 0))
+    (property "Value" "GNDREF" (id 1) (at 160.02 34.29 0))
     (property "Footprint" "" (id 2) (at 158.75 30.48 0)
       (effects (font (size 1.27 1.27)) hide)
